File: chariot-elevateur.sch (EAGLE design)
At the start: 51 parts, among them CON1 XT-60, P1 RG500, Q1 DMN2056U, Q2 DMN2056U, U1 WIZ820IO

Commit message: Update components ref + add debug LEDs + map unused pins for debug
Parts:
- added EXTRA: (no value), pinhead:PINHD-1X5
- added LED4: red, led:LED3MM
- added LED5: orange, led:LED3MM
- added R8, R9: 330, resistor:R-EU_R0805
- AX12_AR, AX12_AV: RS (none) -> 687-8124
- ENCODEUR_DROIT, ENCODEUR_GAUCHE: RS (none) -> 752-1769; RS_F (none) -> 752-1731
- ENDSTOP, JUMPER: RS (none) -> 752-1765; RS_F (none) -> 752-1737
- FUMIGENE: RS (none) -> 688-3283
- LED1: ADAFRUIT (none) -> 879
- LED2: value green -> blue; RS (none) -> 692-1073
- LED3: RS (none) -> 726-9215
- PAS_A_PAS: RS (none) -> 820-1447; RS_F (none) -> 820-1481
- PHARES_AR, PHARES_AV: RS (none) -> 752-1778; RS_F (none) -> 752-1740
- TOF_AR, TOF_AV: RS (none) -> 752-1775; RS_F (none) -> 752-1747
- U1: RS (none) -> 758-1032
Connections:
- new net DEL_ERROR: R8.1, TEENSY.4/CAN0-RX/SDA2/PWM
- new net DEL_WARNING: R9.1, TEENSY.5/PWM
- new net EXTRA_GPIO_1: EXTRA.4, TEENSY.2/PWM
- new net EXTRA_GPIO_2: EXTRA.5, TEENSY.3/CAN0-TX/SCL2/PWM
- new net N$1: LED4.A, R8.2
- new net N$11: LED5.A, R9.2
- net +3V3: now also EXTRA.3
- net +5V/1: now also EXTRA.2
- net GND: now also EXTRA.1, LED4.C, LED5.C
Other:
- moved on the sheet: USB
