File: raspi.brd (EAGLE design)
At the start: 160 x 100 mm, 15 parts

Commit message: shield raspi: shematics done
Parts:
- removed C11, C4: 10µF/50V, resistor:C1210
- removed C9: 220µF/25V, resistor:E3,5-8
- removed D1: DIODE_S15P45, diode_schottky:TO-277A
- removed DC3: TSR 2-2450, dc-dc-converter:SIP3
- removed F1: MF-LSMF300, polyswitch:MF-LSMF300
- removed JP1: (no value), pinhead:1X02
- removed LED1: blue, led:1206
- removed R1: 470, resistor:R0805
- removed RASPPBERRY_PI: (no value), pinhead:2X20/90
- removed S1: (no value), switch:SWITCH_LPV-1
- added ALIM_AUX:C1, ALIM_AUX:C2, ALIM_RPI:C1, ALIM_RPI:C2: 10µF/50V, resistor:C1210
- added ALIM_AUX:C3, ALIM_RPI:C3: 220µF/25V, resistor:E3,5-8
- added ALIM_AUX:D1, ALIM_RPI:D1: SS56B, diode:SMB
- added ALIM_AUX:DC1, ALIM_RPI:DC1: TSR 2-2450, dc-dc-converter:SIP3
- added ALIM_AUX:F1, ALIM_RPI:F1: MF-LSMF300, polyswitch:MF-LSMF300
- added ALIM_AUX:LED1, ALIM_RPI:LED1: blue, led:1206
- added ALIM_AUX:OUTPUT, ALIM_AUX:POWER_INPUT, ALIM_RPI:OUTPUT, ALIM_RPI:POWER_INPUT, PWM: (no value), pinhead:1X02
- added ALIM_AUX:R1, ALIM_RPI:R1: 470, resistor:R0805
- added ALIM_AUX:SJ1, ALIM_RPI:SJ1: (no value), jumper:SJ
- added ALIM_AUX:SW1, ALIM_RPI:SW1: 5MS1S102AM6QES, switch:SPDT_SLIDE_SWITCH
- added I2C, UART: (no value), pinhead:1X04
- added JMP1: 0R-JUMPA, jump-0r-smd:A0R-JMP
- added LIDAR: 05-JST-B5B-XH-A, bt_con-jst-xh:B5B-XH
- added SPI: (no value), pinhead:1X07
- added SV1: (no value), con-lsta:FE20-2
Connections:
- removed net +24V: D1.-, S1.2
- removed net +5V_RPI: RASPPBERRY_PI.2, RASPPBERRY_PI.4
- removed net N$3: LED1.A, R1.1
- removed net N$4: D1.+1, D1.+2, F1.1
- removed net V_LIPO: F1.2, JP1.1
- new net +5V/1: ALIM_AUX:C3.+, ALIM_AUX:DC1.3, ALIM_AUX:OUTPUT.1, ALIM_AUX:R1.2, LIDAR.P$5
- new net ALIM_AUX:N$1: ALIM_AUX:C1.1, ALIM_AUX:C2.1, ALIM_AUX:DC1.1, ALIM_AUX:SJ1.2, ALIM_AUX:SW1.1
- new net ALIM_AUX:N$3: ALIM_AUX:LED1.A, ALIM_AUX:R1.1
- new net ALIM_AUX:N$4: ALIM_AUX:D1.C, ALIM_AUX:SJ1.1, ALIM_AUX:SW1.C
- new net ALIM_AUX:N$6: ALIM_AUX:D1.A, ALIM_AUX:F1.1
- new net ALIM_AUX:N$7: ALIM_AUX:F1.2, ALIM_AUX:POWER_INPUT.2
- new net ALIM_RPI:N$1: ALIM_RPI:C1.1, ALIM_RPI:C2.1, ALIM_RPI:DC1.1, ALIM_RPI:SJ1.2, ALIM_RPI:SW1.1
- new net ALIM_RPI:N$3: ALIM_RPI:LED1.A, ALIM_RPI:R1.1
- new net ALIM_RPI:N$4: ALIM_RPI:D1.C, ALIM_RPI:SJ1.1, ALIM_RPI:SW1.C
- new net ALIM_RPI:N$6: ALIM_RPI:D1.A, ALIM_RPI:F1.1
- new net ALIM_RPI:N$7: ALIM_RPI:F1.2, ALIM_RPI:POWER_INPUT.2
- new net CE0: SPI.6, SV1.24
- new net CE1: SPI.7, SV1.26
- new net MISO: SPI.4, SV1.21
- new net MOSI: SPI.3, SV1.19
- new net PWM0: JMP1.1, PWM.1, SV1.32
- new net PWM1: JMP1.3, PWM.2, SV1.33
- new net RX: LIDAR.P$4, SV1.10, UART.4
- new net SCL: I2C.4, SV1.5
- new net SCLK: SPI.5, SV1.23
- new net SDA: I2C.3, SV1.3
- new net TX: LIDAR.P$3, SV1.8, UART.3
- net +3V3: now also I2C.1, SPI.1, SV1.1, SV1.17, UART.1
- net +5V: now also ALIM_RPI:C3.+, ALIM_RPI:DC1.3, ALIM_RPI:OUTPUT.1, ALIM_RPI:R1.2, SV1.2, SV1.4; no longer C9.+, DC3.3, R1.2
- net GND: now also ALIM_AUX:C1.2, ALIM_AUX:C2.2, ALIM_AUX:C3.-, ALIM_AUX:DC1.2, ALIM_AUX:LED1.C, ALIM_AUX:OUTPUT.2, ALIM_AUX:POWER_INPUT.1, ALIM_AUX:SW1.P$4, ALIM_AUX:SW1.P$5, ALIM_RPI:C1.2, ALIM_RPI:C2.2, ALIM_RPI:C3.-, ALIM_RPI:DC1.2, ALIM_RPI:LED1.C, ALIM_RPI:OUTPUT.2, ALIM_RPI:POWER_INPUT.1, ALIM_RPI:SW1.P$4, ALIM_RPI:SW1.P$5, I2C.2, LIDAR.P$2, SPI.2, SV1.14, SV1.20, SV1.25, SV1.30, SV1.34, SV1.39, SV1.6, SV1.9, UART.2; no longer C11.2, C4.2, C9.-, DC3.2, JP1.2, LED1.C, RASPPBERRY_PI.14, RASPPBERRY_PI.20, RASPPBERRY_PI.25, RASPPBERRY_PI.30, RASPPBERRY_PI.34, RASPPBERRY_PI.39, RASPPBERRY_PI.6, RASPPBERRY_PI.9, S1.B, S1.B1
- net N$1: now also JMP1.2, LIDAR.P$1; no longer C11.1, C4.1, DC3.1, S1.1
- net N$2: now also SV1.29; no longer RASPPBERRY_PI.29
- net N$5: now also SV1.31; no longer RASPPBERRY_PI.31
