File: raspi.sch (EAGLE design)
At the start: 15 parts

Commit message: shield raspi: shematics done
Parts:
- removed C11, C4: 10µF/50V, resistor:C-EUC1210
- removed C9: 220µF/25V, resistor:CPOL-EUE3.5-8
- removed D1: DIODE_S15P45, diode_schottky:DIODE_S15P45
- removed DC3: TSR 2-2450, dc-dc-converter:R-78C5.0-1.0
- removed F1: MF-LSMF300, polyswitch:MF-LSMF300
- removed JP1: (no value), pinhead:PINHD-1X2
- removed LED1: blue, led:LEDSMT1206
- removed R1: 470, resistor:R-EU_R0805
- removed RASPPBERRY_PI: (no value), pinhead:PINHD-2X20/90
- removed S1: (no value), switch:SWITCH_LPV-1
- added I2C, UART: (no value), pinhead:PINHD-1X4
- added JMP1: 0R-JUMPA, jump-0r-smd:0R-JUMPA
- added LIDAR: 05-JST-B5B-XH-A, bt_con-jst-xh:05-JST-B5B-XH-A
- added PWM: (no value), pinhead:PINHD-1X2
- added SPI: (no value), pinhead:PINHD-1X7
- added SV1: (no value), con-lsta:FE20-2
Connections:
- removed net +24V: D1.-, S1.P
- removed net +5V_RPI: RASPPBERRY_PI.2, RASPPBERRY_PI.4
- removed net N$3: LED1.A, R1.1
- removed net N$4: D1.+, F1.1
- removed net V_LIPO: F1.2, JP1.1
- new net +5V/1: LIDAR-5.1
- new net CE0: SPI.6, SV1.24
- new net CE1: SPI.7, SV1.26
- new net MISO: SPI.4, SV1.21
- new net MOSI: SPI.3, SV1.19
- new net PWM0: JMP1-0R.1, PWM.1, SV1.32
- new net PWM1: JMP1-0R.3, PWM.2, SV1.33
- new net RX: LIDAR-4.1, SV1.10, UART.4
- new net SCL: I2C.4, SV1.5
- new net SCLK: SPI.5, SV1.23
- new net SDA: I2C.3, SV1.3
- new net TX: LIDAR-3.1, SV1.8, UART.3
- net +3V3: now also I2C.1, SPI.1, SV1.1, SV1.17, UART.1
- net +5V: now also SV1.2, SV1.4; no longer C9.+, DC3.VOUT, R1.2
- net GND: now also I2C.2, LIDAR-2.1, SPI.2, SV1.14, SV1.20, SV1.25, SV1.30, SV1.34, SV1.39, SV1.6, SV1.9, UART.2; no longer C11.2, C4.2, C9.-, DC3.GND, JP1.2, LED1.C, RASPPBERRY_PI.14, RASPPBERRY_PI.20, RASPPBERRY_PI.25, RASPPBERRY_PI.30, RASPPBERRY_PI.34, RASPPBERRY_PI.39, RASPPBERRY_PI.6, RASPPBERRY_PI.9, S1.B, S1.B1
- net N$1: now also JMP1-0R.2, LIDAR-1.1; no longer C11.1, C4.1, DC3.VIN, S1.O
- net N$2: now also SV1.29; no longer RASPPBERRY_PI.29
- net N$5: now also SV1.31; no longer RASPPBERRY_PI.31
Other:
- moved on the sheet: LED4, R10, R9
