File: chariot-elevateur.brd (EAGLE design)
At the start: 123 x 78 mm, 87 parts, among them P1 RG500, Q1 DMN2056U, Q2 DMN2056U, Q3 DMN2056U, Q4 DMN2056U, U1 WIZ820IO

Commit message: CAM files are ready
Parts:
- added TP4: PTR1PAD1-13, testpad:P1-13
- moved TP3 2.00 mm to (76.0, 10.0)
- renumbered FUMIGENE1 to EXTRA
Connections:
- net +24V: now also TP4.TP
Routing:
- net +24V: track 107.0 -> 110.4 mm
- net SERIAL_AX12_5V: track 149.3 -> 147.3 mm
Other:
- board text added: "12V"
- board text added: "24V"
- board text added: "3.3V"
- board text added: "5V"
- board text added: "5V-EXT"
- board text added: "AX12"
- board text added: "DATA AX12"
- board text added: "DATA F-LED"
- board text added: "DATA R-LED"
- board text added: "ENCODER"
- board text added: "ENDSTOP"
- board text added: "EXTRA"
- board text added: "FRONT LED"
- board text added: "FRONT TOF"
- board text added: "GND"
- board text added: "JUMPER"
- board text added: "REAR LED"
- board text added: "REAR TOF"
- board text added: "SMOKE"
- board text added: "STEPPER"
- board text added: "Teensy 3.5"
- board text added: "USB"
- board text added: "VESC"
- board text added: "error"
- board text added: "pin2"
- board text added: "pin3"
- board text added: "warning"
- board text added: "© 2019 - GobGob Senpaï"
